File: xx-39r-elrs/xx-39r-elrs.kicad_sch (KiCad schematic)
At the start: 47 parts, among them J1 SENSE, J10 PA2, J11 PWR1, J12 PWR2, J13 R_VCC, J14 GND1, J15 GND2, J16 GND3, J2 BAT, J3 M_PORT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

Commit message: Use 0805 for C21/C22
The actual capacitance of the old 0402 might drop below TPS
requirements under load.
Parts:
- C21, C22: footprint Capacitor_SMD:C_0402_1005Metric -> Capacitor_SMD:C_0805_2012Metric
Changed lines of the file:
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@@
 			)
 		)
-		(property "Footprint" "Capacitor_SMD:C_0402_1005Metric"
+		(property "Footprint" "Capacitor_SMD:C_0805_2012Metric"
 			(at 60.96 54.3052 0)
 			(hide yes)
@@
 			)
 		)
-		(property "Footprint" "Capacitor_SMD:C_0402_1005Metric"
+		(property "Footprint" "Capacitor_SMD:C_0805_2012Metric"
 			(at 60.96 65.7352 0)
 			(hide yes)
